Commit message: Working and clean commit

File: bumperbot_description/urdf/bumperbot.urdf.xacro (robot description, xacro)
@@ -192,5 +192,5 @@
   </link>
   <joint name="laser_joint" type="fixed">
-    <origin xyz="-0.0050526 -0.0023221 0.1208" rpy="0 0 3.14" />
+    <origin xyz="-0.0050526 -0.0023221 0.1208" rpy="0 0 0" />
     <parent link="base_link" />
     <child link="laser_link" />

File: bumperbot_description/urdf/bumperbot_gazebo.xacro (robot description, xacro)
@@ -151,5 +151,5 @@
       <plugin name="scan" filename="libgazebo_ros_ray_sensor.so">
         <ros>
-          <remapping>~/out:=scan</remapping>
+          <remapping>~/out:=oscan</remapping>
         </ros>
         <output_type>sensor_msgs/LaserScan</output_type>

File: bumperbot_description/urdf/realsense2.urdf.xacro (robot description, xacro)
@@ -177,6 +177,6 @@
   <plugin name="camera" filename="librealsense_gazebo_plugin.so">
         <prefix>camera</prefix>
-        <depthUpdateRate>30.0</depthUpdateRate>
-        <colorUpdateRate>30.0</colorUpdateRate>
+        <depthUpdateRate>15.0</depthUpdateRate>
+        <colorUpdateRate>15.0</colorUpdateRate>
         <infraredUpdateRate>30.0</infraredUpdateRate>
         <depthTopicName>camera/aligned_depth_to_color/image_raw</depthTopicName>
